File: kicad/controller_board/controller_board.kicad_pcb (KiCad board)
At the start: 2 copper layers, 52.5 x 31 mm, 10 parts, among them J1 Battery Conn, Q1 FQP27P06, SW1 On/Off, SW2 Pair/Direction, U1 ESP32-C3-SuperMini

Commit message: Elininate dead space on right side of controller PCB
Other:
- board size 52.5 x 31 mm -> 49.5 x 31 mm
Changed lines of the file:
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@@
 	(gr_rect
 		(start 149 65)
-		(end 201.5 96)
+		(end 198.5 96)
 		(stroke
 			(width 0.05)
